File: lock_in_amplifier/LNA_test/Power.sch (KiCad schematic (older format))
At the start: 60 parts, among them J1 vref-in, J19 +3V3 OUT, J2 vref, J3 V-IN, J4 GND, J46 -5V OUT, J47 +5V OUT, J5 V+IN, J6 +5V, J7 +3V3, J8 -5V, Q1 DMN640L, Q2 DMN640L, U1 LM833, U2 lm7805, U3 LM7833, U4 lm7905

Commit message: initial lna and power floorplan finished.
Parts:
- U2, U3, U4: footprint TO_SOT_Packages_THT:TO-220_Vertical -> TO_SOT_Packages_THT:TO-220-3_Vertical
Changed lines of the file:
@@
 F 0 "U2" H 5750 1475 50  0000 C CNN
 F 1 "lm7805" H 5900 1475 50  0000 L CNN
-F 2 "TO_SOT_Packages_THT:TO-220_Vertical" H 5900 1575 50  0001 C CIN
+F 2 "TO_SOT_Packages_THT:TO-220-3_Vertical" H 5900 1575 50  0001 C CIN
 F 3 "" H 5900 1300 50  0001 C CNN
 	1    5900 1350
@@
 F 0 "U4" H 5850 4275 50  0000 C CNN
 F 1 "lm7905" H 6000 4275 50  0000 L CNN
-F 2 "TO_SOT_Packages_THT:TO-220_Vertical" H 6000 4375 50  0001 C CIN
+F 2 "TO_SOT_Packages_THT:TO-220-3_Vertical" H 6000 4375 50  0001 C CIN
 F 3 "" H 6000 4100 50  0001 C CNN
 	1    6000 4150
@@
 F 0 "U3" H 5850 2725 50  0000 C CNN
 F 1 "LM7833" H 6000 2725 50  0000 L CNN
-F 2 "TO_SOT_Packages_THT:TO-220_Vertical" H 6000 2825 50  0001 C CIN
+F 2 "TO_SOT_Packages_THT:TO-220-3_Vertical" H 6000 2825 50  0001 C CIN
 F 3 "" H 6000 2550 50  0001 C CNN
 	1    6000 2600
