File: lock_in_amplifier/LIA_Build/PLL.sch (KiCad schematic (older format))
At the start: 71 parts, among them J36 DELAY SEL FINE, J37 DELAY SEL COARSE, U10 74HC4046A, U14 MCP6566, U15 MC74LCX16374, U5 74HC4040, U7 LM833

Commit message: pll finalized - misc cleanup - review candidate
Parts:
- added C60: C, symbol C
- added R105, R106: R, symbol R
- added TP38: C1A, symbol TEST
- added TP39: C1B, symbol TEST
- added TP40: R2, symbol TEST
- added TP41: R1, symbol TEST
- C47: value C -> 100PF
- R74, R75: value R -> 10K
- gave numbers to parts that had none: 7
Connections:
- net GND: now also C60.2
- net at R76.1, R77.1, R84.1: now also R105.2; no longer TP19.1, U10.9 (VCOin)
- net at C47.1, U10.6 (C1A): now also TP38.1
- net at C47.2, U10.7 (C1B): now also TP39.1
- net at R75.1, U10.12 (R2): now also TP40.1
- net at R74.1, U10.11 (R1): now also TP41.1
- net at R84.2, U10.15 (PC3): now also TP26.1
- net at TP28.1: now also R103.2, R104.1, U5.9 (Q0)
- net at R98.2, R99.2, U15.25 (CP1): now also TP32.1
- net at J37.4 (Pin_4), R100.2, R101.2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: now also TP33.1
- net at R104.2, R96.2, R97.2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: now also TP34.1
- net at TP31.1: now also R102.2, R96.1, U5.7 (Q1)
- new net: R105.1, R106.1, TP19.1, U10.9 (VCOin)
- new net: C60.1, R106.2
Other:
- note added: "CENTER FREQUENCY OF 3MHZ\nLOCK RANGE OF 6 MHZ"
- note added: "DIGITAL DELAY DESIGN:\nCOUNTER AT FREUQUENCY HIGHER THAN FMOD.\nSAY 32X (FCLK = 32 X FMOD)\nDELAYS BY N FCLK CYCLES -> DELAY BY N/32 FMOD CYCLES\n\nNEED +- 90 RANGE, 6-10 DEGREE RESOLUTION\nSINE(6) -> 10%\nTHIS WILL PERMIT FULL RANGE (INCLUDING NEGATIVES) OF VALUES.\n\nNOTE THAT YOU HAVE HIGHER FREQUENCIES AVAILABLE \nSO YOU CAN SHIFT THE FVCO TO (SAY) 2X FCLK, AND 128 X FMOD"
- note added: "LOOP FILTER VALUES TBD"
- note added: "PC2 SELECTED FOR DUTY CYCLE IMMUNITY"
- note removed: "DIGITAL DELAY POSSIBILITIES:\nCOUNTER AT FREUQUENCY HIGHER THAN FMOD.\nSAY 64X (FCLK = 64 X FMOD)\nDELAYS BY N FCLK CYCLES -> DELAY BY N/64 FMOD CYCLES\n\nNEED +- 90 RANGE, 6-10 DEGREE RESOLUTION\nSINE(6) -> 10%\nTHIS WILL PERMIT FULL RANGE (INCLUDING NEGATIVES) OF VALUES.\n\nNOTE THAT YOU HAVE HIGHER FREQUENCIES AVAILABLE \nSO YOU CAN SHIFT THE FVCO TO (SAY) 2X FCLK, AND 128 X FMOD"
- note removed: "LOOP FILTER"
- note removed: "SELECT VALUE"
- moved on the sheet: C47, R74, R75

Commit message: started LNA test board.
Parts:
- C45, C46, C47, C48, C49, C50, C51, C52, C53, C56, C57, C58, C59, C60: footprint (none) -> Capacitors_SMD:C_0805
- D8: footprint (none) -> LEDs:LED_0805
- J36: footprint (none) -> Pin_Headers:Pin_Header_Straight_1x10_Pitch2.54mm
- J37: footprint (none) -> Pin_Headers:Pin_Header_Straight_1x05_Pitch2.54mm
- R100, R101, R102, R103, R104, R105, R106, R71, R72, R73, R74, R75, R76, R77, R78, R79, R80, R81, R82, R83, R84, R85, R86, R87, R88, R89, R90, R94, R95, R96, R97, R98, R99: footprint (none) -> Resistors_SMD:R_0805
- TP17, TP18, TP19, TP20, TP21, TP22, TP24, TP25, TP26, TP27, TP28, TP30, TP31, TP32, TP33, TP34, TP35, TP36, TP37, TP38, TP39, TP40, TP41: footprint (none) -> footprints:tyco_RCU_0603_Probe_Pad
- U10: footprint (none) -> Housings_SOIC:SOIC-16_3.9x9.9mm_Pitch1.27mm
- U14: footprint (none) -> TO_SOT_Packages_SMD:SOT-23-5
- U15: footprint (none) -> Housings_SSOP:TSSOP-48_6.1x12.5mm_Pitch0.5mm
- U5: footprint (none) -> Housings_SSOP:TSSOP-16_4.4x5mm_Pitch0.65mm
- U7: footprint (none) -> Housings_SOIC:SO-8_5.3x6.2mm_Pitch1.27mm
