File: lock_in_amplifier/LIA_Build/amplifiers.sch (KiCad schematic (older format))
At the start: 48 parts, among them U1 LM833, U12 LM833, U9 OP1177

Commit message: Added quadrature demod, phase shift to pll
Changed lines of the file:
@@
 $EndComp
 $Comp
-L GND #PWR60
+L GND #PWR059
 U 1 1 5A225760
 P 7050 4350
-F 0 "#PWR60" H 7050 4100 50  0001 C CNN
+F 0 "#PWR059" H 7050 4100 50  0001 C CNN
 F 1 "GND" H 7050 4200 50  0000 C CNN
 F 2 "" H 7050 4350 50  0001 C CNN
@@
 $EndComp
 $Comp
-L GND #PWR56
+L GND #PWR060
 U 1 1 5A2257E8
 P 3200 5250
-F 0 "#PWR56" H 3200 5000 50  0001 C CNN
+F 0 "#PWR060" H 3200 5000 50  0001 C CNN
 F 1 "GND" H 3200 5100 50  0000 C CNN
 F 2 "" H 3200 5250 50  0001 C CNN
@@
 $EndComp
 $Comp
-L GND #PWR58
+L GND #PWR061
 U 1 1 5A22582C
 P 4300 4000
-F 0 "#PWR58" H 4300 3750 50  0001 C CNN
+F 0 "#PWR061" H 4300 3750 50  0001 C CNN
 F 1 "GND" H 4300 3850 50  0000 C CNN
 F 2 "" H 4300 4000 50  0001 C CNN
@@
 $EndComp
 $Comp
-L GND #PWR57
+L GND #PWR062
 U 1 1 5A237D65
 P 3850 6250
-F 0 "#PWR57" H 3850 6000 50  0001 C CNN
+F 0 "#PWR062" H 3850 6000 50  0001 C CNN
 F 1 "GND" H 3850 6100 50  0000 C CNN
 F 2 "" H 3850 6250 50  0001 C CNN
@@
 	3900 4350 3700 4350
 Wire Wire Line
-	3900 3650 3900 3900
-Wire Wire Line
-	3900 3900 3900 4350
-Wire Wire Line
-	6750 4700 7250 4700
-Wire Wire Line
-	7250 4700 7300 4700
+	3900 3650 3900 4350
+Wire Wire Line
+	6750 4700 7300 4700
 Wire Wire Line
 	6750 4050 6750 4700
@@
 	3200 5150 3200 5250
 Wire Wire Line
-	5500 4800 5650 4800
-Wire Wire Line
-	5650 4800 6100 4800
-Wire Wire Line
-	6100 4800 6150 4800
+	5500 4800 6150 4800
 Connection ~ 6100 4800
 Wire Wire Line
@@
 	4750 6150 5100 6150
 Wire Wire Line
-	3650 6250 3850 6250
-Wire Wire Line
-	3850 6250 3950 6250
-Wire Wire Line
-	3950 6250 4150 6250
+	3650 6250 4150 6250
 Connection ~ 3950 6250
 Wire Wire Line
-	3650 5950 3950 5950
-Wire Wire Line
-	3950 5950 4150 5950
+	3650 5950 4150 5950
 Wire Wire Line
 	4150 5950 4150 6050
@@
 	4400 4650 4400 4800
 Wire Wire Line
-	4400 4800 4650 4800
-Wire Wire Line
-	4650 4800 5200 4800
+	4400 4800 5200 4800
 Wire Wire Line
 	5100 6150 5100 4600
 Wire Wire Line
-	5100 4600 5250 4600
-Wire Wire Line
-	5250 4600 6150 4600
+	5100 4600 6150 4600
 Wire Wire Line
 	3700 3850 3700 4050
@@
 	3400 4050 3100 4050
 Wire Wire Line
-	2750 4750 3050 4750
-Wire Wire Line
-	3050 4750 3500 4750
-Wire Wire Line
-	6950 2750 6950 2850
-Wire Wire Line
-	6950 2850 6950 2950
-Wire Wire Line
-	6950 2100 6950 2200
-Wire Wire Line
-	6950 2200 6950 2250
-Wire Wire Line
-	6950 1400 6950 1500
-Wire Wire Line
-	6950 1500 6950 1600
+	2750 4750 3500 4750
+Wire Wire Line
+	6950 2750 6950 2950
+Wire Wire Line
+	6950 2100 6950 2250
+Wire Wire Line
+	6950 1400 6950 1600
 Connection ~ 6950 1500
 Connection ~ 6950 2200
@@
 	6800 1800 6750 1800
 Wire Wire Line
-	6650 1400 6650 1500
-Wire Wire Line
-	6650 1500 6650 1600
-Wire Wire Line
-	6650 2100 6650 2150
-Wire Wire Line
-	6650 2150 6650 2250
-Wire Wire Line
-	6650 2750 6650 2850
-Wire Wire Line
-	6650 2850 6650 2950
+	6650 1400 6650 1600
+Wire Wire Line
+	6650 2100 6650 2250
+Wire Wire Line
+	6650 2750 6650 2950
 Connection ~ 6650 1500
 Connection ~ 6650 2850
@@
 Connection ~ 7250 4700
 Wire Wire Line
-	7250 4700 8850 4700
-Wire Wire Line
-	8850 4700 10100 4700
+	7250 4700 10100 4700
 Text Notes 10200 2900 0    60   ~ 0
 1x2x5x select\n5x\n2x\n1x
 Wire Wire Line
-	9050 1200 9050 1950
-Wire Wire Line
-	9050 1950 9050 2750
-Wire Wire Line
-	9050 2750 9050 2950
-Wire Wire Line
-	9050 2950 9050 3000
-Wire Wire Line
-	9050 3000 9050 3250
+	9050 1200 9050 3250
 Wire Wire Line
 	9050 3250 6950 3250
@@
 Connection ~ 9050 1950
 Wire Wire Line
-	8750 1800 8750 2400
-Wire Wire Line
-	8750 2400 8750 2650
-Wire Wire Line
-	8750 2650 8750 2800
-Wire Wire Line
-	8750 2800 8750 3100
+	8750 1800 8750 3100
 Wire Wire Line
 	8750 1800 7100 1800
@@
 Connection ~ 9050 3000
 Wire Wire Line
-	8450 1500 8450 2200
-Wire Wire Line
-	8450 2200 8450 2550
-Wire Wire Line
-	8450 2550 8450 2850
+	8450 1500 8450 2850
 Wire Wire Line
 	8450 2850 6950 2850
@@
 	5200 1200 6650 1200
 Wire Wire Line
-	5200 3250 5350 3250
-Wire Wire Line
-	5350 3250 6650 3250
+	5200 3250 6650 3250
 Wire Wire Line
 	6300 2550 6650 2550
@@
 	6450 2400 6300 2400
 Wire Wire Line
-	6300 2150 6300 2400
-Wire Wire Line
-	6300 2400 6300 2550
-Wire Wire Line
-	6300 2550 6300 2600
+	6300 2150 6300 2600
 Connection ~ 6300 2550
 Wire Wire Line
@@
 	6150 1950 6650 1950
 Wire Wire Line
-	6150 1500 6150 1800
-Wire Wire Line
-	6150 1800 6150 1950
-Wire Wire Line
-	6150 1950 6150 2400
+	6150 1500 6150 2400
 Wire Wire Line
 	6450 1800 6150 1800
@@
 $EndComp
 $Comp
-L GND #PWR59
+L GND #PWR063
 U 1 1 5A275732
 P 5850 5400
-F 0 "#PWR59" H 5850 5150 50  0001 C CNN
+F 0 "#PWR063" H 5850 5150 50  0001 C CNN
 F 1 "GND" H 5850 5250 50  0000 C CNN
 F 2 "" H 5850 5400 50  0001 C CNN
@@
 Connection ~ 9050 2950
 Wire Wire Line
-	8750 2750 9050 2750
-Wire Wire Line
-	9050 2750 9300 2750
+	8750 2750 9300 2750
 Wire Wire Line
 	8750 2750 8750 2800
@@
 	5200 1200 5200 2250
 Wire Wire Line
-	5200 2750 5200 2850
-Wire Wire Line
-	5200 2850 5200 3100
-Wire Wire Line
-	5200 3100 5200 3250
+	5200 2750 5200 3250
 Connection ~ 5350 3250
 Wire Wire Line
@@
 Connection ~ 6150 2400
 Wire Wire Line
-	4400 2500 4400 3050
-Wire Wire Line
-	4400 3050 4400 3450
+	4400 2500 4400 3450
 Wire Wire Line
 	4400 3450 5650 3450
@@
 	2500 5000 2500 5150
 $Comp
-L GND #PWR55
+L GND #PWR064
 U 1 1 5A257877
 P 2600 5950
-F 0 "#PWR55" H 2600 5700 50  0001 C CNN
+F 0 "#PWR064" H 2600 5700 50  0001 C CNN
 F 1 "GND" H 2600 5800 50  0000 C CNN
 F 2 "" H 2600 5950 50  0001 C CNN
@@
 $EndComp
 $Comp
-L GND #PWR53
+L GND #PWR065
 U 1 1 5A259E13
 P 1600 6050
-F 0 "#PWR53" H 1600 5800 50  0001 C CNN
+F 0 "#PWR065" H 1600 5800 50  0001 C CNN
 F 1 "GND" H 1600 5900 50  0000 C CNN
 F 2 "" H 1600 6050 50  0001 C CNN
@@
 $EndComp
 Wire Wire Line
-	1500 6050 1600 6050
-Wire Wire Line
-	1600 6050 1750 6050
+	1500 6050 1750 6050
 Connection ~ 1600 6050
 Wire Wire Line
-	1400 5750 1500 5750
-Wire Wire Line
-	1500 5750 1750 5750
-Wire Wire Line
-	1750 5750 1850 5750
+	1400 5750 1850 5750
 Connection ~ 1500 5750
 Connection ~ 1750 5750
 Wire Wire Line
-	2150 5750 2250 5750
-Wire Wire Line
-	2250 5750 2400 5750
+	2150 5750 2400 5750
 Wire Wire Line
 	2250 5750 2250 6400
 Wire Wire Line
-	1400 6400 1600 6400
-Wire Wire Line
-	1600 6400 1800 6400
-Wire Wire Line
-	1800 6400 1950 6400
+	1400 6400 1950 6400
 Connection ~ 1800 6400
 Connection ~ 1600 6400
@@
 	1100 5750 850  5750
 $Comp
-L GND #PWR54
+L GND #PWR066
 U 1 1 5A25B123
 P 1700 6700
-F 0 "#PWR54" H 1700 6450 50  0001 C CNN
+F 0 "#PWR066" H 1700 6450 50  0001 C CNN
 F 1 "GND" H 1700 6550 50  0000 C CNN
 F 2 "" H 1700 6700 50  0001 C CNN
@@
 $EndComp
 Wire Wire Line
-	1600 6700 1700 6700
-Wire Wire Line
-	1700 6700 1800 6700
+	1600 6700 1800 6700
 Connection ~ 1700 6700
 Text Notes 950  3450 0    60   ~ 0

Commit message: pll finalized - misc cleanup - review candidate
Connections:
- net GND: now also U12.3 (+), U9.3 (+); no longer S9.1 (B1)
- net at R22.1, S2.2 (A): now also S9.2 (A); no longer U12.2 (-), U9.2 (-)
- net at C44.1, R70.1, S9.3 (B0): now also U12.2 (-), U9.2 (-)
- net at C41.2, R67.2: now also S9.1 (B1)
Other:
- note added: "LM833 / OP1177 SWAPABLE.\nLAYOUT NOTE: \nLAY COMPONENTS ON TOP \nOF EACHOTHER\nONLY POPULATE ONE\nUNSURE HOW TO CLEAR DRC ERROR"
- note removed: "INPUT IMPEDANCE EFFECT ON GAIN OF LNA"
- note removed: "LM833 / OP1177 SWAPABLE.\nLAYOUT NOTE: \nLAY COMPONENTS ON TOP \nOF EACHOTHER\nONLY POPULATE ONE"
- note removed: "SPDT SWITCH\n"
- note removed: "TRADE:\nADD OP AMP AS DEDICATED ACTIVE FILTER\nVS\nUSE NON-INVERTING AMP W/ THIS TOPOLOGY\n\nINVESTIGATE:\nTUNING / ETC."
- moved on the sheet: C30, C41, C42, C43, C44, R22, R53, R54, R67, R68, R69, R70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

Commit message: started LNA test board.
Parts:
- C41, C42, C43, C44: footprint (none) -> Capacitors_SMD:C_0805
- R53, R54, R67, R68, R69, R70: footprint (none) -> Resistors_SMD:R_0805
- TP1, TP2, TP3, TP4: footprint (none) -> footprints:tyco_RCU_0603_Probe_Pad
- U12: footprint (none) -> Housings_SOIC:SO-8_5.3x6.2mm_Pitch1.27mm
Changed lines of the file:
@@
 F 0 "R53" V 6630 5800 50  0000 C CNN
 F 1 "100k" V 6550 5800 50  0000 C CNN
-F 2 "" V 6480 5800 50  0001 C CNN
+F 2 "Resistors_SMD:R_0805" V 6480 5800 50  0001 C CNN
 F 3 "" H 6550 5800 50  0001 C CNN
 	1    6550 5800
@@
 F 0 "R54" V 6630 6100 50  0000 C CNN
 F 1 "100" V 6550 6100 50  0000 C CNN
-F 2 "" V 6480 6100 50  0001 C CNN
+F 2 "Resistors_SMD:R_0805" V 6480 6100 50  0001 C CNN
 F 3 "" H 6550 6100 50  0001 C CNN
 	1    6550 6100
@@
 F 0 "TP2" H 4650 5100 50  0000 C BNN
 F 1 "MID AMP OUT" H 4650 5050 50  0000 C CNN
-F 2 "" H 4650 4800 50  0001 C CNN
+F 2 "footprints:tyco_RCU_0603_Probe_Pad" H 4650 4800 50  0001 C CNN
 F 3 "" H 4650 4800 50  0001 C CNN
 	1    4650 4800
@@
 F 0 "TP3" H 5250 4900 50  0000 C BNN
 F 1 "GAIN AMP REF" H 5250 4850 50  0000 C CNN
-F 2 "" H 5250 4600 50  0001 C CNN
+F 2 "footprints:tyco_RCU_0603_Probe_Pad" H 5250 4600 50  0001 C CNN
 F 3 "" H 5250 4600 50  0001 C CNN
 	1    5250 4600
@@
 F 0 "TP1" H 4400 3350 50  0000 C BNN
 F 1 "END AMP GAIN FB" H 4400 3300 50  0000 C CNN
-F 2 "" H 4400 3050 50  0001 C CNN
+F 2 "footprints:tyco_RCU_0603_Probe_Pad" H 4400 3050 50  0001 C CNN
 F 3 "" H 4400 3050 50  0001 C CNN
 	1    4400 3050
@@
 F 0 "TP4" H 8850 5000 50  0000 C BNN
 F 1 "HIGH GAIN AMP OUT" H 8850 4950 50  0000 C CNN
-F 2 "" H 8850 4700 50  0001 C CNN
+F 2 "footprints:tyco_RCU_0603_Probe_Pad" H 8850 4700 50  0001 C CNN
 F 3 "" H 8850 4700 50  0001 C CNN
 	1    8850 4700
@@
 F 0 "R67" V 2080 4750 50  0000 C CNN
 F 1 "10M" V 2000 4750 50  0000 C CNN
-F 2 "" V 1930 4750 50  0001 C CNN
+F 2 "Resistors_SMD:R_0805" V 1930 4750 50  0001 C CNN
 F 3 "" H 2000 4750 50  0001 C CNN
 	1    2000 4750
@@
 F 0 "R70" V 2830 4750 50  0000 C CNN
 F 1 "10M" V 2750 4750 50  0000 C CNN
-F 2 "" V 2680 4750 50  0001 C CNN
+F 2 "Resistors_SMD:R_0805" V 2680 4750 50  0001 C CNN
 F 3 "" H 2750 4750 50  0001 C CNN
 	1    2750 4750
@@
 F 0 "R68" V 2430 5550 50  0000 C CNN
 F 1 "10M" V 2350 5550 50  0000 C CNN
-F 2 "" V 2280 5550 50  0001 C CNN
+F 2 "Resistors_SMD:R_0805" V 2280 5550 50  0001 C CNN
 F 3 "" H 2350 5550 50  0001 C CNN
 	1    2350 5550
@@
 F 0 "R69" V 2630 5550 50  0000 C CNN
 F 1 "10M" V 2550 5550 50  0000 C CNN
-F 2 "" V 2480 5550 50  0001 C CNN
+F 2 "Resistors_SMD:R_0805" V 2480 5550 50  0001 C CNN
 F 3 "" H 2550 5550 50  0001 C CNN
 	1    2550 5550
@@
 F 0 "C44" H 2875 5500 50  0000 L CNN
 F 1 "270P" H 2875 5300 50  0000 L CNN
-F 2 "" H 2888 5250 50  0001 C CNN
+F 2 "Capacitors_SMD:C_0805" H 2888 5250 50  0001 C CNN
 F 3 "" H 2850 5400 50  0001 C CNN
 	1    2850 5400
@@
 F 0 "C43" H 2525 5000 50  0000 L CNN
 F 1 "270P" H 2525 4800 50  0000 L CNN
-F 2 "" H 2538 4750 50  0001 C CNN
+F 2 "Capacitors_SMD:C_0805" H 2538 4750 50  0001 C CNN
 F 3 "" H 2500 4900 50  0001 C CNN
 	1    2500 4900
@@
 F 0 "C42" H 2275 5000 50  0000 L CNN
 F 1 "270P" H 2275 4800 50  0000 L CNN
-F 2 "" H 2288 4750 50  0001 C CNN
+F 2 "Capacitors_SMD:C_0805" H 2288 4750 50  0001 C CNN
 F 3 "" H 2250 4900 50  0001 C CNN
 	1    2250 4900
@@
 F 0 "C41" H 2025 5500 50  0000 L CNN
 F 1 "270P" H 2025 5300 50  0000 L CNN
-F 2 "" H 2038 5250 50  0001 C CNN
+F 2 "Capacitors_SMD:C_0805" H 2038 5250 50  0001 C CNN
 F 3 "" H 2000 5400 50  0001 C CNN
 	1    2000 5400
@@
 F 0 "U12" H 3800 4850 50  0000 L CNN
 F 1 "LM833" H 3800 4400 50  0000 L CNN
-F 2 "" H 3800 4650 50  0001 C CNN
+F 2 "Housings_SOIC:SO-8_5.3x6.2mm_Pitch1.27mm" H 3800 4650 50  0001 C CNN
 F 3 "" H 3800 4650 50  0001 C CNN
 	1    3800 4650
