File: lock_in_amplifier/pll_test/PLL.sch (KiCad schematic (older format))
At the start: 78 parts, among them J36 DELAY SEL FINE, J37 DELAY SEL COARSE, U10 74HC4046A, U14 MCP6566, U15 MC74LCX16374, U5 74HC4040, U7 LM833

Commit message: misc debug
Parts:
- added TP?: VCO OUT, footprints:tyco_RCU_0603_Probe_Pad, symbol TEST
- U7: footprint Housings_SOIC:SO-8_5.3x6.2mm_Pitch1.27mm -> Housings_SOIC:SOIC-8_3.9x4.9mm_Pitch1.27mm
Other:
- note added: "DNI SELECTORS FOR "STANDARD" \nF / F/64 OPERATION"
Changed lines of the file:
@@
 F 0 "U7" H 3000 1800 50  0000 L CNN
 F 1 "LM833" H 3000 1400 50  0000 L CNN
-F 2 "Housings_SOIC:SO-8_5.3x6.2mm_Pitch1.27mm" H 3000 1600 50  0001 C CNN
+F 2 "Housings_SOIC:SOIC-8_3.9x4.9mm_Pitch1.27mm" H 3000 1600 50  0001 C CNN
 F 3 "" H 3000 1600 50  0001 C CNN
 	2    3000 1600
@@
 	4100 1300 3700 1300
 Wire Wire Line
-	3700 1600 3700 1300
-Wire Wire Line
-	3300 1600 3700 1600
+	3700 1300 3700 1600
+Wire Wire Line
+	3700 1600 3300 1600
 Wire Wire Line
 	4100 1600 4100 1650
@@
 U 1 1 5A296754
 P 7550 4350
-F 0 "R100" V 7630 4350 50  0000 C CNN
+F 0 "R100" V 7550 4150 50  0000 C CNN
 F 1 "0" V 7550 4350 50  0000 C CNN
 F 2 "Resistors_SMD:R_0805" V 7480 4350 50  0001 C CNN
@@
 U 1 1 5A296990
 P 7550 4450
-F 0 "R101" V 7630 4450 50  0000 C CNN
+F 0 "R101" V 7550 4250 50  0000 C CNN
 F 1 "0" V 7550 4450 50  0000 C CNN
 F 2 "Resistors_SMD:R_0805" V 7480 4450 50  0001 C CNN
@@
 U 1 1 5A296FA3
 P 7850 4150
-F 0 "R98" V 7930 4150 50  0000 C CNN
+F 0 "R98" V 7850 3950 50  0000 C CNN
 F 1 "0" V 7850 4150 50  0000 C CNN
 F 2 "Resistors_SMD:R_0805" V 7780 4150 50  0001 C CNN
@@
 U 1 1 5A297067
 P 7850 4250
-F 0 "R99" V 7930 4250 50  0000 C CNN
+F 0 "R99" V 7850 4050 50  0000 C CNN
 F 1 "0" V 7850 4250 50  0000 C CNN
 F 2 "Resistors_SMD:R_0805" V 7780 4250 50  0001 C CNN
@@
 U 1 1 5A297D17
 P 8250 3850
-F 0 "R96" V 8330 3850 50  0000 C CNN
+F 0 "R96" V 8250 3600 50  0000 C CNN
 F 1 "0" V 8250 3850 50  0000 C CNN
 F 2 "Resistors_SMD:R_0805" V 8180 3850 50  0001 C CNN
@@
 U 1 1 5A297DE9
 P 8250 3950
-F 0 "R97" V 8330 3950 50  0000 C CNN
+F 0 "R97" V 8250 3750 50  0000 C CNN
 F 1 "0" V 8250 3950 50  0000 C CNN
 F 2 "Resistors_SMD:R_0805" V 8180 3950 50  0001 C CNN
@@
 Connection ~ 6950 5150
 Wire Wire Line
-	4200 5150 6950 5150
+	6950 5150 4200 5150
 Connection ~ 4200 5150
 Wire Wire Line
@@
 U 1 1 5A29DA5C
 P 8250 3750
-F 0 "R104" V 8330 3750 50  0000 C CNN
+F 0 "R104" V 8250 3500 50  0000 C CNN
 F 1 "0" V 8250 3750 50  0000 C CNN
 F 2 "Resistors_SMD:R_0805" V 8180 3750 50  0001 C CNN
@@
 	4050 5150 4050 4350
 Wire Wire Line
-	4200 3700 4200 5150
+	4200 5150 4200 3700
 Wire Wire Line
 	4200 3700 4050 3700
@@
 Wire Wire Line
 	4150 3600 4050 3600
+Text Notes 7200 3250 0    60   ~ 0
+DNI SELECTORS FOR "STANDARD" \nF / F/64 OPERATION
+Text Notes 7950 4300 0    60   ~ 0
+DNI
+Text Notes 7650 4500 0    60   ~ 0
+DNI
+Text Notes 8350 4000 0    60   ~ 0
+DNI
+Text Notes 8350 3900 0    60   ~ 0
+DNI
+Text Notes 9850 3000 0    60   ~ 0
+DNI
+$Comp
+L TEST TP?
+U 1 1 5A44E8C5
+P 4450 6400
+F 0 "TP?" H 4450 6700 50  0000 C BNN
+F 1 "VCO OUT" H 4450 6650 50  0000 C CNN
+F 2 "footprints:tyco_RCU_0603_Probe_Pad" H 4450 6400 50  0001 C CNN
+F 3 "" H 4450 6400 50  0001 C CNN
+	1    4450 6400
+	1    0    0    -1
+$EndComp
 $EndSCHEMATC
